File: Schematics/LFO-1.kicad_sch (KiCad schematic)
At the start: 66 parts

Commit message: - Updated current libraries - New 7 inc display with ESP32S3 and second USB upload port - Start of I2C feeder interface slave on display.
Parts:
- gave numbers to parts that had none: 54
Connections:
- net at RV14. (3): now also R181.1

Commit message: working interface for 7 inch display with occasional faults.
Connections:
- net at RV14. (3): now also R181.1
Changed lines of the file:
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@@
 	)
 	(symbol
-		(lib_name "Device:R_Potentiometer_US")
 		(lib_id "Device:R_Potentiometer_US")
 		(at 52.07 67.31 270)
@@
 	)
 	(symbol
-		(lib_name "Device:R_Potentiometer_US")
 		(lib_id "Device:R_Potentiometer_US")
 		(at 63.5 36.83 0)
@@
 	)
 	(symbol
-		(lib_name "Device:R_Potentiometer_US")
 		(lib_id "Device:R_Potentiometer_US")
 		(at 115.57 33.02 90)
