File: Schematics/Osc_4_ifc.kicad_sch (KiCad schematic)
At the start: 81 parts, among them J100 Conn_01x12, J101 Conn_01x08, J95 Conn_01x10h, J96 Conn_01x10h, J97 Conn_01x10h, J98 Conn_01x12, J99 Conn_01x12, P3 Conn_01x03, U103 LM358, U106 LM358, U107 LM358, U134 TL074, U136 TL074, U137 TL074, U138 TL074, U139 TL074, U140 LM78L05, U141 LM358, U142 LM358, U143 LM358

Commit message: working interface for 7 inch display with occasional faults.
Connections:
- net at RV26. (3): now also R356.1
Changed lines of the file:
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@@
 	)
 	(symbol
-		(lib_name "Device:R_Potentiometer_US")
 		(lib_id "Device:R_Potentiometer_US")
 		(at 67.945 48.895 270)
@@
 	)
 	(symbol
-		(lib_name "Device:R_Potentiometer_US")
 		(lib_id "Device:R_Potentiometer_US")
 		(at 176.53 48.895 270)
@@
 	)
 	(symbol
-		(lib_name "Device:R_Potentiometer_US")
 		(lib_id "Device:R_Potentiometer_US")
 		(at 285.75 48.895 270)
