File: Schematics/Noise.kicad_sch (KiCad schematic)
At the start: 74 parts, among them J81 Conn_01x04, J82 Conn_01x04, J83 Conn_01x02, J84 Conn_01x04, J85 Conn_01x02, J86 Conn_01x04, J87 Conn_01x04, J88 Conn_01x04, J89 Conn_01x03, Q10 BC547, Q7 BC547, Q8 BC547, Q9 BC547, U122 TL074, U123 ADG419BN, U124 TL074, U125 TL074, U126 LM78L05

Commit message: Prelude to split configurations.
Parts:
- removed J81, J82, J84, J86, J87, J88: Conn_01x04, symbol Connector_keyed_kicad_sym:Conn_01x04
- removed J83, J85: Conn_01x02, symbol Connector_keyed_kicad_sym:Conn_01x02
- removed Q10, Q7, Q8, Q9: BC547, Package_TO_SOT_THT:TO-92_Inline, symbol Transistor_BJT:BC547
- removed R253, R256, R259: 20k, symbol Device:R_Small_US
- removed R254, R255, R257, R258: 10k, symbol Device:R_Small_US
- removed R260: 267, symbol Device:R_Small_US
- removed RV16: 100k, symbol Device:R_Potentiometer_US
- removed RV17: 2k, symbol Device:R_Potentiometer_US
- removed U122, U124, U125: TL074, symbol Amplifier_Operational:TL074
- removed U123: ADG419BN, Package_DIP:DIP-8_W7.62mm, symbol Analog_Switch:ADG419BN
- removed VR3: TL431A, digikey-footprints:TO-92-3_Formed_Leads, symbol dk_PMIC-Voltage-Reference:TL431CLPM
- added C141, C146, C147, C148, C83: 0.1µF, symbol Device:C_Small
- added C144, C145: .1µF, symbol Device:C_Small
- added C31: 1µF, symbol Device:C_Polarized_Small_US
- added C84: 22pF, symbol Device:C_Small
- added J81, J82, J83, J84: Conn_01x02, symbol My Connectors:Conn_01x02
- added J85, J86: Conn_01x03, symbol My Connectors:Conn_01x03
- added JP6, JP7, JP8: Jumper_2_Small_Open, symbol Jumper:Jumper_2_Small_Open
- added Q1: 2N3904, Package_TO_SOT_THT:TO-92_Inline, symbol Transistor_BJT:2N3904
- added Q2, Q7: BSS138, digikey-footprints:SOT-23-3, symbol dk_Transistors-FETs-MOSFETs-Single:BSS138
- added R167, R198, R202: 470k, symbol Device:R_Small_US
- added R199, R203, R204, R207, R208, R211, R214, R215, R216, R217, R218, R221, R222: 10k, symbol Device:R_Small_US
- added R200: 2M, symbol Device:R_Small_US
- added R201, R210: 100k, symbol Device:R_Small_US
- added R205, R209, R212: 15k, symbol Device:R_Small_US
- added R206, R213: 220k, symbol Device:R_Small_US
- added R219, R220, R223, R224: 10K, symbol Device:R_Small_US
- added RV10: 100k, symbol Device:R_Potentiometer_US
- added U63, U67, U70, U74, U75, U76: TL074, symbol My Chips:TL074
- added U64: TL072, symbol Amplifier_Operational:TL072
- added U65, U66, U68, U69: DG212C, symbol My Chips:DG212C
- added U71: PCF8575, Package_SO:SSOP-24_5.3x8.2mm_P0.65mm, symbol Interface_Expansion:PCF8575DBR
- added U73: LM1117-3.3, symbol Regulator_Linear:LM1117-3.3
- C109: value 0.22µF -> 0.1µF
- C110, C111, C118: value 2.2µF -> 0.1µF
- C112: value 5.0µF -> 0.22µF
- C113, C116: value 100pF -> 0.1µF
- C114, C117: value 0.15µF -> 0.1µF
- C115: value 0.033µF -> 0.1µF
- R225, R226, R234, R238, R239: value 10k -> 10K
- R227: value 200K -> 10K
- R228: value 100k -> 10K
- R229: value 470 -> 10K
- R230: value 3.3k -> 10K
- R231: value 20k -> 10K
- R232: value 4.7m -> 10K
- R233: value 470K -> 10K
- R235, R236: value 560k -> 10K
- R237: value 1k -> 10K
- R240, R241: value 30k -> 10k
- R242, R250: value 20k -> 10k
- R243: value 3.3M -> 10k
- R244: value 3.3k -> 10k
- R245: value 220 -> 10k
- R246: value 420 -> 10k
- R248: value 49.9k -> 10k
- U126: value LM78L05 -> LM1117-5
Connections:
- net +2V5 is gone; now on an unnamed net: R248.2
- net To Mixer is gone; now on net +3.3V: R237.2
- net +12V: now also C114.2, C116.2, C122.2, C141.2, C146.1, C147.1, R167.1, U63.4 (V+), U64.8 (V+), U65.13 (V+), U66.13 (V+), U67.4 (V+), U68.13 (V+), U69.13 (V+), U70.4 (V+); no longer R227.1, R228.1, R229.1, R230.1
- net -12V: now also C113.1, C115.1, C117.1, C118.1, C148.2, R199.2, U63.11 (V-), U64.4 (V-), U65.4 (V-), U66.4 (V-), U67.11 (V-), U68.4 (V-), U69.4 (V-), U70.11 (V-); no longer C109.2, C116.2, C118.2, R243.2, R244.2, R245.2, R246.2
- net GNDA: now also C111.2, C112.2, C144.2, C145.2, C146.2, C147.2, C148.1, C31.2, J81.2 (Pin_2), J82.2 (Pin_2), J83.2 (Pin_2), J84.2 (Pin_2), J85.1 (Pin_1), J86.3 (Pin_3), JP6.1 (A), JP7.1 (A), JP8.1 (A), R200.2, R201.2, R205.1, R209.1, R212.1, U63.10 (+), U71.12 (GND), U73.1 (GND); no longer C122.2, R241.2
- net at R247.2: now also R245.2, R246.2, U75.5 (+); no longer R250.1
- net at R249.2: now also R250.2, R251.2, R252.2, U76.5 (+); no longer R247.1
- net at R251.1: now also U68.10 (D3); no longer R252.2
- net at R249.1: now also U68.2 (D1)
- net +3.3V: now reaches R226.1
- net +3.3V: now also R225.2, R227.2, R228.1, R229.2, R230.1, R231.2, R232.1, R233.2, R234.1, R235.2, R236.1, R238.1, R239.2, C145.1, Q2.1, Q7.1, R219.1, R220.1, R221.2, R222.2, R223.1, R224.1, U65.12 (VL), U66.12 (VL), U68.12 (VL), U69.12 (VL), U71.24 (VCC), U73.2 (VO)
- net NB4: now reaches R225.1
- net NB4: now also U68.8 (IN4), U71.20 (P17); no longer R226.2
- net NW4: now reaches R231.1
- net NW4: now also U68.1 (IN1), U71.17 (P14); no longer R225.2
- net at C110.1: now also R204.1, RV10. (3), U63.8, U67.10 (+); no longer R235.2
- net at R240.1: now also C110.2, U64.3 (+); no longer C111.2
- net at R241.1: now also U66.2 (D1); no longer C117.2
- net at R242.1: now also U66.15 (D2); no longer R238.2
- net NW3: now reaches R239.1
- net NW3: now also U69.1 (IN1), U71.13 (P10)
- net at R244.1: now also U66.7 (D4); no longer C114.2
- net at C112.1: now also R208.2, U63.5 (+); no longer R232.2
- net at R252.1: now also U68.7 (D4)
- net at R246.1: now also U69.15 (D2)
- net NP3: now reaches R237.1
- net NP3: now also U69.16 (IN2), U71.14 (P11)
- net at R245.1: now also U69.2 (D1); no longer C115.2
- net at R248.1: now also U69.7 (D4)
- net +5VA: no longer names the net of C121.1, U126.1 (VO)
- net +5VA: now also C144.1, U73.3 (VI); no longer C122.1
- new net: Q7.2, R222.1, U71.23 (SDA)
- new net: JP6.2 (B), R219.2, U71.21 (A0)
- new net: C83.2, R200.1, U63.12 (+)
- new net: C84.1, R201.1, R202.1, U63.13 (-)
- new net: C109.1, C84.2, R202.2, U63.14
- new net: C113.2, C114.1, U65.5 (GND)
- new net: JP7.2 (B), R220.2, U71.2 (A1)
- new net: JP8.2 (B), R223.2, U71.3 (A2)
- new net: R213.2, R214.1, U64.1
- new net: R212.2, R213.1, U64.2 (-)
- new net: R209.2, R210.1, U63.6 (-)
- new net: R210.2, R211.1, U63.7
- new net: C118.2, C141.1, U69.5 (GND)
- new net: J84.1 (Pin_1), U76.6 (-), U76.7
- new net: R214.2, U67.12 (+)
- new net: R247.1, U69.10 (D3)
- new net: R206.2, R207.1, R208.1, U63.1
- new net: C31.1, R167.2, R198.1
- new net: R243.1, U66.10 (D3)
- new net: R241.2, R242.2, R243.2, R244.2, U70.5 (+)
- new net: R216.1, U65.10 (D3)
- new net: R215.2, R216.2, R217.2, R218.2, U74.5 (+)
- new net: C83.1, Q1.1 (E), R198.2
- new net: C115.2, C116.1, U66.5 (GND)
- new net: C117.2, C122.1, U68.5 (GND)
- new net: R215.1, U65.15 (D2)
- new net: R218.1, U65.2 (D1)
- new net: R217.1, U65.7 (D4)
- new net: R211.2, U67.5 (+)
- new net: J81.1 (Pin_1), U74.6 (-), U74.7
- new net: R250.1, U68.15 (D2)
- new net: Q2.2, R221.1, U71.22 (SCL)
- new net: R205.2, R206.1, U63.2 (-)
- new net: C111.1, R204.2, U63.3 (+)
- new net: R203.2, RV10. (3), U63.9 (-)
- new net: R207.2, U67.3 (+)
- new net: J82.1 (Pin_1), U75.6 (-), U75.7
- new net: J83.1 (Pin_1), U70.6 (-), U70.7
- new net: Q1.2 (B), R199.1
- new net: C109.2, R203.1
- new net Blue: U65.6 (S4), U66.6 (S4), U67.13 (-), U67.14, U68.6 (S4), U69.6 (S4)
- new net NB1: R230.2, U65.8 (IN4), U71.7 (P3)
- new net NB2: R238.2, U66.8 (IN4), U71.11 (P7)
- new net NB3: R233.1, U69.8 (IN4), U71.16 (P13)
- new net NP1: R226.2, U65.16 (IN2), U71.5 (P1)
- new net NP2: R234.2, U66.16 (IN2), U71.9 (P5)
- new net NP4: R229.1, U68.16 (IN2), U71.18 (P15)
- new net NR1: R228.2, U65.9 (IN3), U71.6 (P2)
- new net NR2: R236.2, U66.9 (IN3), U71.10 (P6)
- new net NR3: R235.1, U69.9 (IN3), U71.15 (P12)
- new net NR4: R227.1, U68.9 (IN3), U71.19 (P16)
- new net NW1: R224.2, U65.1 (IN1), U71.4 (P0)
- new net NW2: R232.2, U66.1 (IN1), U71.8 (P4)
- new net Pink: U65.14 (S2), U66.14 (S2), U67.1, U67.2 (-), U68.14 (S2), U69.14 (S2)
- new net Red: U65.11 (S3), U66.11 (S3), U67.6 (-), U67.7, U68.11 (S3), U69.11 (S3)
- new net SCL0: J85.3 (Pin_3), J86.1 (Pin_1), Q2.3
- new net SDA0: J85.2 (Pin_2), J86.2 (Pin_2), Q7.3
- new net White: U65.3 (S1), U66.3 (S1), U67.8, U67.9 (-), U68.3 (S1), U69.3 (S1)
Other:
- note added: "A0"
- note added: "A1"
- note added: "A2"
- note added: "LEVEL"
- note added: "NC"
- note removed: "Noise Generator"
- note removed: "Output"
- note removed: "Pink"
- note removed: "Selector"
- note removed: "White"
- title: Noise Generator and Mixer -> Noise Generator and Multiplexer
- moved on the sheet: C119, C120, C121, C123, C124, C125, J89, U126
