File: Schematics/Noise.kicad_sch (KiCad schematic)
At the start: 116 parts, among them J207 Conn_01x03, J219 Conn_01x03, J222 Conn_01x03, J275 Conn_01x02, J276 Conn_01x02, J296 Conn_01x02, J297 Conn_01x02, Q29 2N3904, Q36 BSS138, Q37 BSS138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

Commit message: Fixed schematic errors.
Connections:
- net SCL0: no longer names the net of J219.1 (Pin_1), J222.3 (Pin_3), Q36.3
- net SDA0: no longer names the net of J219.2 (Pin_2), J222.2 (Pin_2), Q37.3
Other:
- moved on the sheet: J219, J222
