File: Schematics/Osc2_Carry.kicad_sch (KiCad schematic)
At the start: 55 parts, among them J40 Conn_01x04, J41 Conn_01x02, J42 Conn_01x02, J43 Screw_Terminal_01x03, J44 Screw_Terminal_01x03, J45 Conn_01x04, U21 MCP4728, U22 MCP4728, U23 TL072, U24 LM358, U25 LM358, U26 LME49720N, U27 TL072, U28 LM1117-5, U29 MCP4728, U30 MCP4728, U31 LM358

Commit message: More features and fixes.
Parts:
- R12, R25: value 22.1k -> 12k
Other:
- note added: "0-8V"
- note added: "Note 1: Adjust for C0 to C8"
- note added: "[Note 1]"
- note removed: "0-10V"
Changed lines of the file:
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@@
 		)
 	)
+	(text "Note 1: Adjust for C0 to C8"
+		(exclude_from_sim no)
+		(at 279.146 181.102 0)
+		(effects
+			(font
+				(size 1.5748 1.5748)
+			)
+			(justify left top)
+		)
+	)
 	(text "_{TRIM}"
 		(exclude_from_sim no)
@@
 		)
 	)
+	(text "[Note 1]"
+		(exclude_from_sim no)
+		(at 312.674 29.972 0)
+		(effects
+			(font
+				(size 1.27 1.27)
+			)
+		)
+	)
 	(text "Osc #1"
 		(exclude_from_sim no)
@@
 		)
 	)
+	(text "[Note 1]"
+		(exclude_from_sim no)
+		(at 167.894 29.21 0)
+		(effects
+			(font
+				(size 1.27 1.27)
+			)
+		)
+	)
 	(text "+12V"
 		(exclude_from_sim no)
@@
 		)
 	)
-	(text "0-10V"
+	(text "0-8V"
 		(exclude_from_sim no)
 		(at 158.242 28.194 0)
@@
 		)
 	)
-	(text "0-10V"
+	(text "0-8V"
 		(exclude_from_sim no)
 		(at 303.022 28.194 0)
@@
 			)
 		)
-		(property "Value" "22.1k"
+		(property "Value" "12k"
 			(at 149.606 32.004 0)
 			(effects
@@
 			)
 		)
-		(property "Value" "22.1k"
+		(property "Value" "12k"
 			(at 294.386 32.004 0)
 			(effects
