File: Schematics/3PoleStateVarVCF.kicad_sch (KiCad schematic)
At the start: 168 parts, among them J54 Conn_01x04, J55 Conn_01x03, J56 Conn_01x04, J57 Conn_01x04, U238 PCF8574, U239 LM78L05, U242 AMS1117-3.3, U270 DG212C, U277 DG212C, U32 SSI2164, U33 TL072, U34 TL074, U35 TL074, U36 TL074, U37 TL072, U38 TL074, U39 SSI2164, U40 MCP4728, U41 TL072, U42 TL072, U43 TL072

Commit message: Updated schematics.  Added modulation control to VCF.
Parts:
- renumbered D18 to D?, U43 to U?, U36 to U?, U35 to U?, U38 to U?, U37 to U?, U33 to U?, U34 to U?, U42 to U?, U41 to U?
Connections:
- net +12V: no longer U?.4 (V+), U?.4 (V+), U?.4 (V+), U?.4 (V+), U?.8 (V+), U?.8 (V+), U?.8 (V+), U?.8 (V+)
- net -12V: no longer U?.11 (V-), U?.11 (V-), U?.11 (V-), U?.11 (V-), U?.4 (V-), U?.4 (V-), U?.4 (V-), U?.4 (V-)
- net GNDA: now also U?.1, U?.3 (+), U?.3 (+), U?.3 (+), U?.3 (+), U?.3 (+), U?.3 (+), U?.3 (+), U?.3 (+); no longer U?.10 (+), U?.10 (+), U?.5 (+), U?.5 (+), U?.5 (+), U?.5 (+), U?.5 (+), U?.5 (+)
- net at C64.1, R41.1, R43.1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: now also U?.1; no longer U?.14
- net at C75.2, R73.2, R76.1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: now also U?.3 (+); no longer U?.5 (+)
- net at C77.2, R78.1, R79.2: now also U?.1, U?.3 (+); no longer U?.10 (+), U?.7
- net at R71.1, R78.2: now also U?.2 (-); no longer U?.13 (-)
- net at C71.2, R61.1, U39.11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: now also U?.1; no longer U?.7
- net at C79.1, U39.12: now also U?.2 (-); no longer U?.9 (-)
- net at C96.2, J57.2 (Pin_2), R97.1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: now also U?.1; no longer U?.7
- net at C65.2, R47.2, R50.1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: now also U?.3 (+); no longer U?.5 (+)
- net at C70.2, R55.1: now also U?.1, U?.3 (+); no longer U?.12 (+), U?.8
- net at C77.1, U39.5: now also U?.2 (-); no longer U?.6 (-)
- net at C96.1, R86.1, R87.1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: now also U?.2 (-); no longer U?.6 (-)
- net at R36.1, R38.1, R41.2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: now also U?.2 (-); no longer U?.6 (-)
- net at R33.2, R36.2: now also U?.1; no longer U?.7
- net at C79.2, R81.1: now also U?.1, U?.3 (+); no longer U?.12 (+), U?.8
- net at C67.2, R52.1, R53.2: now also U?.1, U?.3 (+); no longer U?.10 (+), U?.7
- net at R48.1, R50.2: now also U?.3 (+); no longer U?.12 (+)
- net at R45.1, R52.2: now also U?.2 (-); no longer U?.13 (-)
- net at C70.1, U32.12: now also U?.2 (-); no longer U?.9 (-)
- net at C71.1, R30.1, R57.1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: now also U?.2 (-); no longer U?.6 (-)
- net at C67.1, U32.5: now also U?.2 (-); no longer U?.6 (-)
- net at R62.1, R64.1, R67.2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: now also U?.2 (-); no longer U?.6 (-)
- net at R59.2, R62.2: now also U?.1; no longer U?.7
- net at C74.1, R67.1, R69.1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: now also U?.1; no longer U?.14
- net at R74.1, R76.2: now also U?.3 (+); no longer U?.12 (+)
- new net: U270.14 (S2), U?.1, U?.2 (-)
- new net: U270.11 (S3), U?.1, U?.2 (-)
- new net: U270.6 (S4), U?.1, U?.2 (-)
- new net: U277.11 (S3), U?.1, U?.2 (-)
- new net: U277.14 (S2), U?.1, U?.2 (-)
- new net: U277.6 (S4), U?.1, U?.2 (-)

Commit message: Updated schematics and added low pass filter and new filter mux.
Parts:
- removed U? (x9): TL072, symbol Amplifier_Operational:TL072
- removed U? (x13): TL074, symbol Amplifier_Operational:TL074
- removed U? (x8): TL074, symbol My Chips:TL074
- added U38, U41, U42: TL072, symbol Amplifier_Operational:TL072
- added U43, U52, U53, U54: TL074, symbol My Chips:TL074
Connections:
- net +12V: now also U38.8 (V+), U41.8 (V+), U42.8 (V+), U43.4 (V+), U52.4 (V+), U53.4 (V+), U54.4 (V+)
- net -12V: now also U38.4 (V-), U41.4 (V-), U42.4 (V-), U43.11 (V-), U52.11 (V-), U53.11 (V-), U54.11 (V-)
- net GNDA: now also U38.3 (+), U38.5 (+), U41.3 (+), U41.5 (+), U42.3 (+), U42.5 (+), U43.10 (+), U43.3 (+), U43.5 (+), U52.10 (+), U52.3 (+), U52.5 (+)
- net at C64.1, R41.1, R43.1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: now also U43.14
- net at R63.1, R65.2: now also U41.1, U54.3 (+)
- net at R56.1, R59.1, R63.2: now also U41.2 (-)
- net at C55.1, R27.1, R28.1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: now also U42.2 (-)
- net at C75.2, R73.2, R76.1: now also U52.1, U54.5 (+)
- net at C75.1, U39.4: now also U52.2 (-)
- net at C77.2, R78.1, R79.2: now also U52.7, U54.10 (+)
- net at R71.1, R78.2: now also U52.13 (-)
- net at C71.2, R61.1, U39.11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: now also U42.7
- net at C79.1, U39.12: now also U52.9 (-)
- net at U270.14 (S2): now also U53.6 (-), U53.7
- net at C65.2, R47.2, R50.1: now also U43.1, U53.5 (+)
- net at C70.2, R55.1: now also U43.8, U53.12 (+)
- net at U270.11 (S3): now also U53.8, U53.9 (-)
- net at U270.3 (S1): now also U53.1, U53.2 (-)
- net at U270.6 (S4): now also U53.13 (-), U53.14
- net at C77.1, U39.5: now also U52.6 (-)
- net at C55.2, R35.1, U32.11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: now also U42.1
- net at R33.2, R36.2: now also U38.7
- net at R36.1, R38.1, R41.2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: now also U38.6 (-)
- net at C65.1, U32.4: now also U43.2 (-)
- net at C79.2, R81.1: now also U52.8, U54.12 (+)
- net at U277.11 (S3): now also U54.8, U54.9 (-)
- net at U277.14 (S2): now also U54.6 (-), U54.7
- net at U277.3 (S1): now also U54.1, U54.2 (-)
- net at U277.6 (S4): now also U54.13 (-), U54.14
- net at C67.2, R52.1, R53.2: now also U43.7, U53.10 (+)
- net at R45.1, R52.2: now also U43.13 (-)
- net at R48.1, R50.2: now also U43.12 (+)
- net at C70.1, U32.12: now also U43.9 (-)
- net at C71.1, R30.1, R57.1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: now also U42.6 (-)
- net at C67.1, U32.5: now also U43.6 (-)
- net at R62.1, R64.1, R67.2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: now also U41.6 (-)
- net at R32.1, R33.1, R37.2: now also U38.2 (-)
- net at R59.2, R62.2: now also U41.7
- net at C74.1, R67.1, R69.1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: now also U52.14
- net at R37.1, R39.2: now also U38.1, U53.3 (+)
- net at R74.1, R76.2: now also U52.12 (+)
