File: Schematics/LowPassFilter.kicad_sch (KiCad schematic)
At the start: 57 parts, among them U37 TL072, U56 SSI2140, U58 TL072, U59 TL072, U60 TL072

Commit message: Updated schematics, adding new low pass fillter and, added some statistical synth data to monitor.
Parts:
- R356: value 18k -> 20k
- R359: value 12k -> 22.1k
Other:
- note added: "Note 1: Adjust for +5.00v to -5.00v"
- note added: "[Note 1]"
- moved on the sheet: C128, C129, R341, U56F
