File: Schematics/OutputMIX.kicad_sch (KiCad schematic)
At the start: 118 parts, among them J205 Conn_01x04, J208 Conn_01x04, J221 Conn_01x03, J231 Conn_01x04, J232 Conn_01x04, J235 Conn_01x04, J236 Conn_01x04, J238 Conn_01x04, J241 Conn_01x04, J242 Conn_01x04, J244 Conn_01x04, J249 Conn_01x04, J250 Conn_01x04, J251 Conn_01x04, J252 Conn_01x04, J253 Conn_01x04, J254 Conn_01x04, J269 Conn_01x02, J74 Conn_01x04, U221 LM1117-5, U243 PCF8574, U246 LM1117-3.3, U280 DG212C, U281 DG212C, U44 MCP4728, U45 TL074, U46 TL074, U47 TL074, U48 TL074, U49 SSI2164, U50 TL074, U51 TL072

Commit message: Updated schematics.  Added modulation control to VCF.
Other:
- moved on the sheet: C323, C324, C325, C326, C353, C379, U221, U246, U45E, U46E, U47E, U48E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

Commit message: Updated schematics and added low pass filter and new filter mux.
Parts:
- added J270: Conn_01x02, symbol My Connectors:Conn_01x02
- added R837: 49.9k, symbol Device:R_Small_US
Connections:
- net GND: now also J270.2 (Pin_2)
- net at C107.1, R830.1, U50.9 (-): now also R837.2
- net Osc1 renamed LP1
- net Osc2 renamed LP2
- net Osc3 renamed LP3
- net Osc4 renamed LP4
- net Osc5 renamed LP5
- net Osc6 renamed LP6
- net Osc7 renamed LP7
- net Osc8 renamed LP8
- new net: J270.1 (Pin_1), R837.1
Other:
- note added: "3 State Filter Input"
- note added: "LP VCF Input"
- note added: "Low Pass switch"
- note removed: "Filter Input"
- note removed: "Oscillator switch"

Commit message: Corrected audio I/O on many schematics and added date to them.  Minor tweaks in voice interfaces.
Connections:
- net Flt1: now also U45.8, U45.9 (-); no longer U45.13 (-)
- net Flt2: now also U45.13 (-), U45.14; no longer U45.8, U45.9 (-)
- net Flt3: now also U46.8, U46.9 (-); no longer U46.13 (-), U46.14
- net Flt4: now also U46.13 (-), U46.14; no longer U46.8, U46.9 (-)
- net Flt5: now also U47.8, U47.9 (-); no longer U47.13 (-), U47.14
- net Flt6: now also U47.13 (-), U47.14; no longer U47.8, U47.9 (-)
- net Flt7: now also U48.8, U48.9 (-); no longer U48.13 (-), U48.14
- net Flt8: now also U48.13 (-), U48.14; no longer U48.8, U48.9 (-)
- net LP1: now also U45.1, U45.2 (-); no longer U45.6 (-), U45.7
- net LP2: now also U45.6 (-), U45.7; no longer U45.1, U45.2 (-)
- net LP3: now also U46.1, U46.2 (-); no longer U46.6 (-), U46.7
- net LP4: now also U46.6 (-), U46.7; no longer U46.1, U46.2 (-)
- net LP5: now also U47.1, U47.2 (-); no longer U47.7
- net LP6: now also U47.6 (-), U47.7; no longer U47.1, U47.2 (-)
- net LP7: now also U48.1, U48.2 (-); no longer U48.6 (-), U48.7
- net LP8: now also U48.6 (-), U48.7; no longer U48.1, U48.2 (-)
- net at J241.4 (Pin_4), J244.1 (Pin_1): now also U47.5 (+)
Other:
- moved on the sheet: J241, J244, J249, J250, U45B, U46A, U46B, U46C, U46D, U47A, U47B, U48A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
