File: Schematics/SpareBoards/Oscc_6Ifc.kicad_sch (KiCad schematic)
At the start: 95 parts, among them J52 Conn_01x10h, J53 Conn_01x10h, J54 Conn_01x10h, J55 Conn_01x10h, J56 Conn_01x12, J57 Conn_01x12, J58 Conn_01x12, J59 Conn_01x12, J60 Conn_01x04, J61 Conn_01x10h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

Commit message: updated schematics.
Connections:
- net at RV6. (3): now also R145.1
- net at RV7. (3): now also R146.1
- net at RV8. (3): now also R147.1
Changed lines of the file:
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@@
 		(fields_autoplaced yes)
 		(property "Reference" "U106"
-			(at 70.3252 53.2846 0)
+			(at 68.072 53.086 0)
 			(effects
 				(font
 					(size 0.889 0.889)
 				)
+				(justify left)
 			)
 		)
 		(property "Value" "LM358"
-			(at 71.12 54.61 0)
+			(at 68.072 54.356 0)
 			(effects
 				(font
 					(size 0.889 0.889)
 				)
+				(justify left)
 			)
 		)
@@
 			)
 		)
-		(property "Description" ""
+		(property "Description" "Low-Power, Dual Operational Amplifiers, DIP-8/SOIC-8/TO-99-8"
 			(at 67.31 57.15 0)
 			(effects
@@
 	)
 	(symbol
+		(lib_name "LM358_3")
 		(lib_id "Amplifier_Operational:LM358")
 		(at 227.33 57.15 0)
@@
 		(fields_autoplaced yes)
 		(property "Reference" "U107"
-			(at 226.06 55.8799 0)
+			(at 228.346 53.34 0)
 			(effects
 				(font
-					(size 1.27 1.27)
+					(size 0.889 0.889)
 				)
 				(justify left)
-				(hide yes)
 			)
 		)
 		(property "Value" "LM358"
-			(at 226.06 57.1499 0)
+			(at 228.346 54.61 0)
 			(effects
 				(font
-					(size 1.27 1.27)
+					(size 0.889 0.889)
 				)
 				(justify left)
-				(hide yes)
 			)
 		)
@@
 			)
 		)
-		(property "Description" ""
+		(property "Description" "Low-Power, Dual Operational Amplifiers, DIP-8/SOIC-8/TO-99-8"
 			(at 227.33 57.15 0)
 			(effects
@@
 	)
 	(symbol
+		(lib_name "LM358_2")
 		(lib_id "Amplifier_Operational:LM358")
 		(at 227.33 30.48 0)
@@
 		(fields_autoplaced yes)
 		(property "Reference" "U103"
-			(at 226.06 29.2099 0)
+			(at 228.092 26.162 0)
 			(effects
 				(font
-					(size 1.27 1.27)
+					(size 0.889 0.889)
 				)
 				(justify left)
-				(hide yes)
 			)
 		)
 		(property "Value" "LM358"
-			(at 226.06 30.4799 0)
+			(at 228.092 27.432 0)
 			(effects
 				(font
-					(size 1.27 1.27)
+					(size 0.889 0.889)
 				)
 				(justify left)
-				(hide yes)
 			)
 		)
@@
 			)
 		)
-		(property "Description" ""
+		(property "Description" "Low-Power, Dual Operational Amplifiers, DIP-8/SOIC-8/TO-99-8"
 			(at 227.33 30.48 0)
 			(effects
