File: Schematics/SpareBoards/LFO-1.kicad_sch (KiCad schematic)
At the start: 54 parts, among them J66 Conn_01x04, J67 Conn_01x04, J68 Conn_01x10h, J69 Conn_01x03, U114 LM324, U115 LM324, U116 SSI2130, U117 LM324, U118 LM78L05

Commit message: Current State with updated LFO for original board.
Parts:
- removed unit 5 of U115
Connections:
- net at RV14. (3): now also R181.1
